Commit message: New robot description

File: catkin_ws/src/simulation/urdf/arm.urdf (robot description, URDF)
Before this commit: robot myfirst, 3 links, 2 joints
Links:
- added link forearm; visual cylinder length=0.35 radius=0.04
- added link upper_arm; visual cylinder length=0.3 radius=0.04
Joints:
- added joint t2: type revolute, parent shoulder, child upper_arm, origin xyz=0 0 0.3 rpy=-1.570796 0 0, axis 0 0 1, limit lower=0.0 upper=0.548 effort=1000.0 velocity=0.5
- added joint t3: type revolute, parent upper_arm, child forearm, origin xyz=0.35 0 0 rpy=0 0 0, axis 0 0 1, limit lower=0.0 upper=0.548 effort=1000.0 velocity=0.5

Commit message: Functional urdf file

File: catkin_ws/src/simulation/urdf/arm.urdf (robot description, URDF)
Before this commit: robot myfirst, 5 links, 4 joints
Joints:
- joint t1: axis 0 0 1 -> 0 1 0; limit lower=0.0 upper=0.548 effort=1000.0 velocity=0.5 -> lower=0.0 upper=3.14159265 effort=1000.0 velocity=0.5
- joint t2: axis 0 0 1 -> 0 -1 0; limit lower=0.0 upper=0.548 effort=1000.0 velocity=0.5 -> lower=-1.570796 upper=1.570796 effort=1000.0 velocity=0.5
- joint t3: limit lower=0.0 upper=0.548 effort=1000.0 velocity=0.5 -> lower=-1.570796 upper=1.570796 effort=1000.0 velocity=0.5; origin xyz=0.35 0 0 rpy=0 0 0 -> xyz=0 0 0 rpy=0 0 0
